File: guitar-amp.kicad_pcb (KiCad board)
At the start: 2 copper layers, 44 parts, among them J1 AudioJack3_Switch, U1 ECC81, U2 ECC81, U3 EL84

Commit message: Model the schematic
Parts:
- removed J1: AudioJack3_Switch, Connector_Audio:Jack_6.35mm_Neutrik_NMJ6HFD2-AU_Horizontal
- removed U1, U2: ECC81, Valve:Valve_Noval_P
- removed U3: EL84, Valve:Valve_Noval_P
- added D1: Bridge Rectifier, Diode_THT:Diode_Bridge_32.0x5.6x17.0mm_P10.0mm_P7.5mm, F.Cu at (22.0, 174.0)
- added F1: Fuse, Fuse:Fuseholder_Cylinder-5x20mm_Schurter_0031_8201_Horizontal_Open, F.Cu at (19.0, 160.0)
- added J2: Input, Connector_Audio:Jack_6.35mm_Neutrik_NMJ6HFD2-AU_Horizontal, F.Cu at (15.1, 141.9)
- added V1: ECC81, Valve:Valve_Noval_P, F.Cu at (102.8, 164.0)
- added V2: ECC81, Valve:Valve_Noval_P, F.Cu at (114.0, 140.3)
- added V3: EL84, Valve:Valve_Noval_P, F.Cu at (79.1, 161.6)
- added VR1: 1M, Potentiometer_THT:Potentiometer_Piher_PT-15-V15_Vertical, F.Cu at (139.1, 136.6)
- added VR2: 1M, Potentiometer_THT:Potentiometer_Piher_PT-15-V15_Vertical, F.Cu at (128.0, 153.2)
- added VR4: 1M Log, Potentiometer_THT:Potentiometer_Piher_PT-15-V15_Vertical, F.Cu at (109.0, 160.3)
- added VR6: 1M, Potentiometer_THT:Potentiometer_Piher_PT-15-V15_Vertical, F.Cu at (120.2, 136.6)
- C10, C9: value 22n -> 1u
- C12: value 50u -> 100u / 25V
- R1: value R -> 10k
- R10: value R -> 68k
- R11, R12, R15, R17: value R -> 470k
- R13: value R -> 1M
- R14: value R -> 2.7k
- R16: value R -> 1.2k
- R18: value R -> 820
- R19: value R -> 130
- R2, R4: value R -> 1k
- R20: value R -> 100 / 2W
- R21, R5, R6, R7: value R -> 100k
- R22, R23: value R -> 100
- R8: value R -> 33k
- R9: value R -> 5.6k
- moved VR3 31.4 mm to (41.9, 91.2)
Connections:
- C1 pad 1: unconnected-(C1-Pad1) -> Net-(R5-Pad1)
- C1 pad 2: unconnected-(C1-Pad2) -> GND
- C10 pad 1: unconnected-(C10-Pad1) -> Net-(C10-Pad1)
- C10 pad 2: unconnected-(C10-Pad2) -> GND
- C11 pad 1: unconnected-(C11-Pad1) -> Net-(V1-Pad8)
- C11 pad 2: unconnected-(C11-Pad2) -> GND
- C12 pad 1: unconnected-(C12-Pad1) -> Net-(C12-Pad1)
- C12 pad 2: unconnected-(C12-Pad2) -> GND
- C13 pad 1: unconnected-(C13-Pad1) -> Net-(C13-Pad1)
- C13 pad 2: unconnected-(C13-Pad2) -> GND
- C14 pad 1: unconnected-(C14-Pad1) -> Net-(R2-Pad2)
- C14 pad 2: unconnected-(C14-Pad2) -> GND
- C15 pad 1: unconnected-(C15-Pad1) -> Net-(C15-Pad1)
- C15 pad 2: unconnected-(C15-Pad2) -> Net-(V1-Pad7)
- C2 pad 1: unconnected-(C2-Pad1) -> Net-(R1-Pad2)
- C2 pad 2: unconnected-(C2-Pad2) -> GND
- C3 pad 1: unconnected-(C3-Pad1) -> Net-(V2-Pad3)
- C3 pad 2: unconnected-(C3-Pad2) -> Net-(C3-Pad2)
- C4 pad 1: unconnected-(C4-Pad1) -> Net-(V1-Pad6)
- C4 pad 2: unconnected-(C4-Pad2) -> Net-(VR1-Pad1)
- C5 pad 1: unconnected-(C5-Pad1) -> Net-(V1-Pad1)
- C5 pad 2: unconnected-(C5-Pad2) -> Net-(C5-Pad2)
- C6 pad 1: unconnected-(C6-Pad1) -> Net-(C8-Pad1)
- C6 pad 2: unconnected-(C6-Pad2) -> Net-(C6-Pad2)
- C7 pad 1: unconnected-(C7-Pad1) -> Net-(VR1-Pad2)
- C7 pad 2: unconnected-(C7-Pad2) -> Net-(R11-Pad2)
- C8 pad 1: unconnected-(C8-Pad1) -> Net-(C8-Pad1)
- C8 pad 2: unconnected-(C8-Pad2) -> Net-(C8-Pad2)
- C9 pad 1: unconnected-(C9-Pad1) -> Net-(R16-Pad1)
- C9 pad 2: unconnected-(C9-Pad2) -> GND
- R1 pad 1: unconnected-(R1-Pad1) -> Net-(R5-Pad1)
- R1 pad 2: unconnected-(R1-Pad2) -> Net-(R1-Pad2)
- R10 pad 1: unconnected-(R10-Pad1) -> Net-(R13-Pad1)
- R10 pad 2: unconnected-(R10-Pad2) -> Net-(C15-Pad1)
- R11 pad 1: unconnected-(R11-Pad1) -> Net-(VR1-Pad2)
- R11 pad 2: unconnected-(R11-Pad2) -> Net-(R11-Pad2)
- R12 pad 1: unconnected-(R12-Pad1) -> Net-(R12-Pad1)
- R12 pad 2: unconnected-(R12-Pad2) -> Net-(R12-Pad2)
- R13 pad 1: unconnected-(R13-Pad1) -> Net-(R13-Pad1)
- R13 pad 2: unconnected-(R13-Pad2) -> GND
- R14 pad 1: unconnected-(R14-Pad1) -> Net-(V1-Pad8)
- R14 pad 2: unconnected-(R14-Pad2) -> GND
- R15 pad 1: unconnected-(R15-Pad1) -> Net-(R11-Pad2)
- R15 pad 2: unconnected-(R15-Pad2) -> GND
- R16 pad 1: unconnected-(R16-Pad1) -> Net-(R16-Pad1)
- R16 pad 2: unconnected-(R16-Pad2) -> GND
- R17 pad 1: unconnected-(R17-Pad1) -> Net-(R12-Pad2)
- R17 pad 2: unconnected-(R17-Pad2) -> GND
- R18 pad 1: unconnected-(R18-Pad1) -> Net-(C10-Pad1)
- R18 pad 2: unconnected-(R18-Pad2) -> GND
- R19 pad 1: unconnected-(R19-Pad1) -> Net-(C12-Pad1)
- R19 pad 2: unconnected-(R19-Pad2) -> GND
- R2 pad 1: unconnected-(R2-Pad1) -> Net-(R1-Pad2)
- R2 pad 2: unconnected-(R2-Pad2) -> Net-(R2-Pad2)
- R20 pad 1: unconnected-(R20-Pad1) -> Net-(C13-Pad1)
- R20 pad 2: unconnected-(R20-Pad2) -> Net-(R2-Pad2)
- R21 pad 1: unconnected-(R21-Pad1) -> GND
- R21 pad 2: unconnected-(R21-Pad2) -> Net-(R2-Pad2)
- R22 pad 1: unconnected-(R22-Pad1) -> Net-(C12-Pad1)
- R22 pad 2: unconnected-(R22-Pad2) -> Net-(V2-Pad4)
- R23 pad 1: unconnected-(R23-Pad1) -> Net-(C12-Pad1)
- R23 pad 2: unconnected-(R23-Pad2) -> Net-(V3-Pad5)
- R3 pad 1: unconnected-(R3-Pad1) -> Net-(R1-Pad2)
- R3 pad 2: unconnected-(R3-Pad2) -> Net-(V2-Pad2)
- R4 pad 1: unconnected-(R4-Pad1) -> Net-(R1-Pad2)
- R4 pad 2: unconnected-(R4-Pad2) -> Net-(R4-Pad2)
- R5 pad 1: unconnected-(R5-Pad1) -> Net-(R5-Pad1)
- R5 pad 2: unconnected-(R5-Pad2) -> Net-(V1-Pad6)
- R6 pad 1: unconnected-(R6-Pad1) -> Net-(R5-Pad1)
- R6 pad 2: unconnected-(R6-Pad2) -> Net-(C5-Pad2)
- R7 pad 1: unconnected-(R7-Pad1) -> Net-(V2-Pad3)
- R7 pad 2: unconnected-(R7-Pad2) -> GND
- R8 pad 1: unconnected-(R8-Pad1) -> Net-(V2-Pad3)
- R8 pad 2: unconnected-(R8-Pad2) -> Net-(C8-Pad1)
- R9 pad 1: unconnected-(R9-Pad1) -> Net-(R9-Pad1)
- R9 pad 2: unconnected-(R9-Pad2) -> Net-(VR6-Pad2)
- VR3 pad 1: unconnected-(VR3-Pad1) -> Net-(C6-Pad2)
- VR3 pad 2: unconnected-(VR3-Pad2) -> Net-(VR3-Pad2)
- VR3 pad 3: unconnected-(VR3-Pad3) -> Net-(C3-Pad2)
- VR5 pad 1: unconnected-(VR5-Pad1) -> GND
- VR5 pad 2: unconnected-(VR5-Pad2) -> Net-(C8-Pad2)
- VR5 pad 3: unconnected-(VR5-Pad3) -> Net-(VR5-Pad3)

Commit message: Roughly layout the components on the PCB
Parts:
- removed F1: Fuse, Fuse:Fuseholder_Cylinder-5x20mm_Schurter_0031_8201_Horizontal_Open
- added J1: Speaker Output, TerminalBlock_RND:TerminalBlock_RND_205-00001_1x02_P5.00mm_Horizontal, F.Cu at (242.9, 59.3)
- added J3: AC Mains, TerminalBlock_RND:TerminalBlock_RND_205-00002_1x03_P5.00mm_Horizontal, F.Cu at (126.0, 50.7)
- added J4: Screw_Terminal_01x02, TerminalBlock_RND:TerminalBlock_RND_205-00001_1x02_P5.00mm_Horizontal, F.Cu at (138.5, 50.5)
- added J5: Screw_Terminal_01x02, TerminalBlock_RND:TerminalBlock_RND_205-00001_1x02_P5.00mm_Horizontal, F.Cu at (166.5, 50.5)
- added J6: Screw_Terminal_01x02, TerminalBlock_RND:TerminalBlock_RND_205-00001_1x02_P5.00mm_Horizontal, F.Cu at (149.5, 50.5)
- added R24: R, Resistor_THT:R_Axial_Power_L20.0mm_W6.4mm_P25.40mm, F.Cu at (176.0, 43.3)
- added SW1: SW_SPST, Button_Switch_THT:SW_CuK_JS202011CQN_DPDT_Straight, F.Cu at (185.3, 53.4)
- added T1: Transformer_1P_1S, TerminalBlock_RND:TerminalBlock_RND_205-00003_1x04_P5.00mm_Horizontal, F.Cu at (220.8, 59.3)
- D1: value Bridge Rectifier -> Bridge Rectifier GBU 6M; footprint Diode_THT:Diode_Bridge_32.0x5.6x17.0mm_P10.0mm_P7.5mm -> Diode_THT:Diode_Bridge_Vishay_GBU
- V1, V2, V3: footprint Valve:Valve_Noval_P -> Valve:Valve_ECC-83-1
- VR1, VR2, VR4, VR6: footprint Potentiometer_THT:Potentiometer_Piher_PT-15-V15_Vertical -> Potentiometer_THT:Potentiometer_Alps_RK163_Single_Horizontal
- moved R19 210.1 mm to (246.4, 98.0), turned to -90 degrees
- moved R9 204.8 mm to (234.6, 127.0)
- moved R22 192.6 mm to (246.4, 94.8), turned to 90 degrees
- moved R23 191.4 mm to (242.4, 94.8), turned to 90 degrees
- moved VR3 181.5 mm to (217.8, 135.9), turned to 90 degrees
- moved R7 177.2 mm to (222.2, 127.0), turned to 180 degrees
- moved D1 174.5 mm to (155.0, 61.1), turned to 90 degrees
- moved VR5 173.6 mm to (198.5, 135.9), turned to 90 degrees
- moved R2 172.9 mm to (201.4, 99.3), turned to 90 degrees
- moved V3 166.0 mm to (232.8, 99.0)
- moved R4 162.9 mm to (207.0, 104.0)
- moved R8 159.2 mm to (210.4, 92.2), turned to -90 degrees
- moved R20 157.3 mm to (200.2, 62.3)
- moved R21 140.9 mm to (199.9, 57.3)
- moved R3 138.7 mm to (206.4, 99.8), turned to 90 degrees
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Connections:
- net GND renamed Earth
Other:
- board outline added: 160 x 100 mm
- board text added: "TODO: - Softstart switch which footprint? - Softstart resistor which size / footprint?"

Commit message: First draft of routing
Parts:
- moved T1 25.8 mm to (246.5, 60.5), turned to 180 degrees
- moved D1 19.1 mm to (165.3, 77.2)
- moved J1 18.5 mm to (224.4, 60.5), turned to 180 degrees
- moved R1 17.0 mm to (165.0, 119.0)
- moved J3 14.0 mm to (136.0, 60.5)
- moved J5 14.0 mm to (176.5, 60.3)
- moved C15 13.9 mm to (133.0, 102.5)
- moved J4 13.7 mm to (148.0, 60.3)
- moved J6 13.7 mm to (159.0, 60.3)
- moved R24 11.9 mm to (181.3, 54.0), turned to 0 degrees
- moved R14 11.8 mm to (124.0, 98.4)
- moved SW1 11.3 mm to (185.0, 64.7)
- moved C5 10.4 mm to (161.0, 107.5), turned to -90 degrees
- moved C11 9.60 mm to (124.0, 95.0)
- moved C13 2.81 mm to (195.5, 76.8)
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Connections:
- net Net-(C1-Pad1) renamed /HighDC_227VDC
- net Net-(C13-Pad1) renamed /HighDC_Prefilter
- net Net-(C14-Pad1) renamed /HighDC_Post
- net Net-(C2-Pad1) renamed /HighDC_241VDC
- net Net-(C3-Pad1) renamed /HighDC_143VDC
- net Net-(C5-Pad1) renamed /HighDC_V1B_Anode
- net Net-(D1-Pad2) renamed /HighDC_Trafo1
- net Net-(D1-Pad3) renamed /HighDC_Trafo2
- net Net-(J3-Pad1) renamed /AC_L
- net Net-(J3-Pad2) renamed /AC_N
- net Net-(R3-Pad2) renamed /HighDC_V2A_Anode
- net Net-(R4-Pad2) renamed /HighDC_GateValve3
- net Net-(T1-Pad1) renamed /HighDC_OT
Routing:
- net Net-(R22-Pad2): track 0.00 -> 182.2 mm, vias 0 -> 4
- net Net-(J5-Pad1): track 0.00 -> 176.1 mm, vias 0 -> 4
- net /HighDC_Post: track 0.00 -> 69.0 mm
- net /HighDC_143VDC: track 0.00 -> 65.5 mm
- net /HighDC_241VDC: track 0.00 -> 60.0 mm
- net Net-(C6-Pad2): track 0.00 -> 50.1 mm
- net /HighDC_Prefilter: track 0.00 -> 50.0 mm
- net /HighDC_OT: track 0.00 -> 43.0 mm
- net Net-(C4-Pad1): track 0.00 -> 40.5 mm
- net Net-(R12-Pad1): track 0.00 -> 40.3 mm, vias 0 -> 2
- net /HighDC_227VDC: track 0.00 -> 38.6 mm
- net Net-(C6-Pad1): track 0.00 -> 35.7 mm
- net Net-(C7-Pad2): track 0.00 -> 32.7 mm
- net Net-(R9-Pad1): track 0.00 -> 31.3 mm
- net /HighDC_V2A_Anode: track 0.00 -> 25.7 mm
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- added copper zone on B.Cu, net Earth
Other:
- board size 160 x 100 mm -> 135 x 90 mm
- board text removed: "TODO: - Softstart switch which footprint? - Softstart resistor which size / footprint?"

Commit message: Routing improvements
Parts:
- added H1: MountingHole, MountingHole:MountingHole_3.2mm_M3, F.Cu at (122.0, 67.0)
- added H2: MountingHole, MountingHole:MountingHole_3.2mm_M3, F.Cu at (245.0, 74.0)
- added H3: MountingHole, MountingHole:MountingHole_3.2mm_M3, F.Cu at (245.0, 119.0)
- added H4: MountingHole, MountingHole:MountingHole_3.2mm_M3, F.Cu at (122.0, 112.0)
- added R8: 33k, Resistor_THT:R_Axial_DIN0207_L6.3mm_D2.5mm_P7.62mm_Horizontal, F.Cu at (210.4, 92.2)
- C12: footprint Capacitor_THT:CP_Radial_D6.3mm_P2.50mm -> Capacitor_THT:CP_Radial_D8.0mm_P3.80mm
- moved R7 6.45 mm to (225.0, 121.2), turned to 90 degrees
- moved J3 5.50 mm to (136.0, 55.0)
- moved J5 5.33 mm to (176.0, 55.0)
- moved J4 5.30 mm to (148.0, 55.0)
- moved J6 5.30 mm to (159.0, 55.0)
- moved R17 4.00 mm to (167.0, 92.4)
- moved R12 2.23 mm to (170.0, 100.0)
- moved C12 1.39 mm to (240.0, 105.0), turned to -90 degrees
- moved C3 1.39 mm to (225.0, 127.0)
- moved R18 1.19 mm to (175.4, 92.8)
- moved C10 1.07 mm to (175.0, 96.0)
- moved R19 1.00 mm to (246.4, 99.0)
- moved R4 0.17 mm to (207.0, 103.8)
Routing:
- net Earth: track 11.8 -> 0.00 mm
- net /HighDC_Trafo2: track 10.6 -> 15.9 mm
- net /HighDC_Trafo1: track 18.3 -> 23.7 mm
- net Net-(J5-Pad1): track 176.1 -> 181.2 mm
- net /HighDC_143VDC: track 65.5 -> 62.5 mm
- net Net-(C6-Pad1): track 35.7 -> 38.3 mm
- net Net-(R12-Pad1): track 40.3 -> 37.9 mm
- net Net-(J5-Pad2): track 21.6 -> 20.0 mm
- net Net-(R12-Pad2): track 16.2 -> 17.7 mm
- net /AC_N: track 24.7 -> 25.5 mm
- net Net-(C12-Pad1): track 24.7 -> 25.5 mm
- net /HighDC_227VDC: track 38.6 -> 37.8 mm
- net Net-(C3-Pad2): track 10.4 -> 9.81 mm
- net Net-(C7-Pad2): track 32.7 -> 33.2 mm
