File: preamp/preamp.kicad_pcb (KiCad board)
At the start: 2 copper layers, 69.1 x 23.9 mm, 18 parts, among them J1 XLR3_AudioJack2_Combo, J2 AudioJack2, J3 AudioJack2, U1 SSM2019

Commit message: milling
Parts:
- moved C2 13.7 mm to (106.4, 77.0), turned to 180 degrees
- moved H2 12.3 mm to (169.0, 63.0)
Other:
- board size 69.1 x 23.9 mm -> 66.1 x 23.9 mm
Changed lines of the file:
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@@
   )
   (footprint "MountingHole:MountingHole_3.2mm_M3_DIN965" (layer "F.Cu")
-    (at 162.052 73.152)
+    (at 169 63)
     (descr "Mounting Hole 3.2mm, no annular, M3, DIN965")
     (tags "mounting hole 3.2mm no annular m3 din965")
@@
   )
   (footprint "Capacitor_THT:C_Disc_D3.0mm_W1.6mm_P2.50mm" (layer "F.Cu")
-    (at 97.536 87.376 -90)
+    (at 106.390757 76.98756 180)
     (descr "C, Disc series, Radial, pin pitch=2.50mm, , diameter*width=3.0*1.6mm^2, Capacitor, http://www.vishay.com/docs/45233/krseries.pdf")
     (tags "C Disc series Radial pin pitch 2.50mm  diameter 3.0mm width 1.6mm Capacitor")
@@
     (property "Sheetname" "")
     (attr through_hole)
-    (fp_text reference "C2" (at 1.25 -2.05 90) (layer "F.SilkS")
-      (effects (font (size 1 1) (thickness 0.15)))
-    )
-    (fp_text value "100p" (at 1.25 2.05 90) (layer "F.Fab")
-      (effects (font (size 1 1) (thickness 0.15)))
-    )
-    (fp_text user "${REFERENCE}" (at 1.25 0 90) (layer "F.Fab")
+    (fp_text reference "C2" (at 1.25 -2.05) (layer "F.SilkS")
+      (effects (font (size 1 1) (thickness 0.15)))
+    )
+    (fp_text value "100p" (at 1.25 2.05) (layer "F.Fab")
+      (effects (font (size 1 1) (thickness 0.15)))
+    )
+    (fp_text user "${REFERENCE}" (at 1.25 0) (layer "F.Fab")
       (effects (font (size 0.6 0.6) (thickness 0.09)))
     )
@@
     (fp_line (start -0.25 -0.8) (end -0.25 0.8) (layer "F.Fab") (width 0.1))
     (fp_line (start 2.75 0.8) (end 2.75 -0.8) (layer "F.Fab") (width 0.1))
-    (pad "1" thru_hole oval (at 0 0) (size 3 2) (drill 0.8) (layers *.Cu *.Mask)
+    (pad "1" thru_hole oval (at 0 0 270) (size 3 2) (drill 0.8) (layers *.Cu *.Mask)
       (net 3 "Net-(C2-Pad1)") (pintype "passive"))
-    (pad "2" thru_hole circle (at 2.5 0 270) (size 1.6 1.6) (drill 0.8) (layers *.Cu *.Mask)
+    (pad "2" thru_hole circle (at 2.5 0 180) (size 1.6 1.6) (drill 0.8) (layers *.Cu *.Mask)
       (net 2 "GNDA") (pintype "passive"))
     (model "${KICAD6_3DMODEL_DIR}/Capacitor_THT.3dshapes/C_Disc_D3.0mm_W1.6mm_P2.50mm.wrl"
@@
     )
   )
-  (gr_rect (start 95.504 74.168) (end 164.592 98.044) (layer "Edge.Cuts") (width 0.1) (fill none))
+  (gr_rect (start 98.504 74.168) (end 164.592 98.044) (layer "Edge.Cuts") (width 0.1) (fill none))
   (gr_text "XLR Preamp  - v1.1 - 3.5.2023" (at 119.38 97.028) (layer "F.SilkS")
     (effects (font (size 1.2 1.2) (thickness 0.25)))
@@
   (segment (start 112.268 77.216) (end 109.982 79.502) (width 0.8) (layer "B.Cu") (net 1))
   (segment (start 122.428 81.788) (end 124.968 81.788) (width 0.8) (layer "B.Cu") (net 3))
-  (segment (start 98.552 87.376) (end 97.536 87.376) (width 0.8) (layer "B.Cu") (net 3))
-  (segment (start 100.584 85.344) (end 98.552 87.376) (width 0.8) (layer "B.Cu") (net 3))
+  (segment (start 101.563 84.365) (end 100.584 85.344) (width 0.8) (layer "B.Cu") (net 3))
+  (segment (start 106.390757 76.98756) (end 106.390757 84.354243) (width 0.8) (layer "B.Cu") (net 3))
+  (segment (start 106.390757 84.354243) (end 106.38 84.365) (width 0.8) (layer "B.Cu") (net 3))
+  (segment (start 106.38 84.365) (end 101.563 84.365) (width 0.8) (layer "B.Cu") (net 3))
   (segment (start 126.1872 83.0072) (end 128.524 83.0072) (width 0.8) (layer "B.Cu") (net 3))
   (segment (start 124.968 81.788) (end 126.1872 83.0072) (width 0.8) (layer "B.Cu") (net 3))
-  (segment (start 97.536 87.376) (end 103.262823 87.376) (width 0.8) (layer "B.Cu") (net 3))
   (segment (start 122.428 85.852) (end 122.428 81.788) (width 0.8) (layer "B.Cu") (net 3))
   (segment (start 106.172 84.466823) (end 110.097177 88.392) (width 0.8) (layer "B.Cu") (net 3))
-  (segment (start 103.262823 87.376) (end 106.172 84.466823) (width 0.8) (layer "B.Cu") (net 3))
   (segment (start 110.097177 88.392) (end 119.888 88.392) (width 0.8) (layer "B.Cu") (net 3))
   (segment (start 119.888 88.392) (end 122.428 85.852) (width 0.8) (layer "B.Cu") (net 3))
