File: preamp/preamp.kicad_pcb (KiCad board)
At the start: 2 copper layers, 66.1 x 23.9 mm, 18 parts, among them J1 XLR3_AudioJack2_Combo, J2 AudioJack2, J3 AudioJack2, U1 SSM2019

Commit message: Small changes
Parts:
- moved C6 1.50 mm to (122.8, 83.3)
Routing:
- net Net-(C2-Pad1): track 43.0 -> 40.9 mm
Changed lines of the file:
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@@
   )
   (footprint "Package_DIP:DIP-8_W7.62mm_LongPads" (layer "F.Cu")
-    (at 128.524 77.9272)
+    (at 128.499658 77.956753)
     (descr "8-lead though-hole mounted DIP package, row spacing 7.62 mm (300 mils), LongPads")
     (tags "THT DIP DIL PDIP 2.54mm 7.62mm 300mil LongPads")
@@
   )
   (footprint "Capacitor_THT:C_Disc_D3.0mm_W1.6mm_P2.50mm" (layer "F.Cu")
-    (at 122.428 81.788 90)
+    (at 122.768362 83.251972 90)
     (descr "C, Disc series, Radial, pin pitch=2.50mm, , diameter*width=3.0*1.6mm^2, Capacitor, http://www.vishay.com/docs/45233/krseries.pdf")
     (tags "C Disc series Radial pin pitch 2.50mm  diameter 3.0mm width 1.6mm Capacitor")
@@
     (effects (font (size 1.2 1.2) (thickness 0.25)))
   )
+  (segment (start 122.768362 80.751972) (end 122.768362 79.984362) (width 0.8) (layer "B.Cu") (net 1))
+  (segment (start 122.768362 80.751972) (end 123.037791 80.482543) (width 0.8) (layer "B.Cu") (net 1))
+  (segment (start 110.102177 80.772) (end 122.748334 80.772) (width 0.8) (layer "B.Cu") (net 1))
+  (segment (start 123.037791 80.482543) (end 128.485448 80.482543) (width 0.8) (layer "B.Cu") (net 1))
+  (segment (start 122.768362 79.984362) (end 120 77.216) (width 0.8) (layer "B.Cu") (net 1))
+  (segment (start 112.268 77.216) (end 109.982 79.502) (width 0.8) (layer "B.Cu") (net 1))
   (segment (start 109.982 80.651823) (end 110.102177 80.772) (width 0.8) (layer "B.Cu") (net 1))
-  (segment (start 125.1204 80.4672) (end 128.524 80.4672) (width 0.8) (layer "B.Cu") (net 1))
-  (segment (start 122.428 79.288) (end 122.072 79.288) (width 0.8) (layer "B.Cu") (net 1))
-  (segment (start 123.9412 79.288) (end 125.1204 80.4672) (width 0.8) (layer "B.Cu") (net 1))
-  (segment (start 117.9576 80.772) (end 119.4416 79.288) (width 0.8) (layer "B.Cu") (net 1))
-  (segment (start 119.4416 79.288) (end 122.428 79.288) (width 0.8) (layer "B.Cu") (net 1))
-  (segment (start 122.072 79.288) (end 120 77.216) (width 0.8) (layer "B.Cu") (net 1))
-  (segment (start 122.428 79.288) (end 123.9412 79.288) (width 0.8) (layer "B.Cu") (net 1))
-  (segment (start 110.102177 80.772) (end 117.9576 80.772) (width 0.8) (layer "B.Cu") (net 1))
+  (segment (start 128.485448 80.482543) (end 128.499658 80.496753) (width 0.8) (layer "B.Cu") (net 1))
   (segment (start 109.982 79.502) (end 109.982 80.651823) (width 0.8) (layer "B.Cu") (net 1))
-  (segment (start 112.268 77.216) (end 109.982 79.502) (width 0.8) (layer "B.Cu") (net 1))
-  (segment (start 109.883991 88.178814) (end 120.101186 88.178814) (width 0.8) (layer "B.Cu") (net 3))
-  (segment (start 122.428 81.788) (end 124.968 81.788) (width 0.8) (layer "B.Cu") (net 3))
+  (segment (start 122.748334 80.772) (end 122.768362 80.751972) (width 0.8) (layer "B.Cu") (net 1))
+  (segment (start 122.428 83.592334) (end 122.768362 83.251972) (width 0.8) (layer "B.Cu") (net 3))
+  (segment (start 122.768362 83.251972) (end 123.013134 83.0072) (width 0.8) (layer "B.Cu") (net 3))
+  (segment (start 106.172 84.466823) (end 109.883991 88.178814) (width 0.8) (layer "B.Cu") (net 3))
   (segment (start 106.390757 76.98756) (end 106.390757 84.354243) (width 0.8) (layer "B.Cu") (net 3))
   (segment (start 106.390757 84.354243) (end 106.38 84.365) (width 0.8) (layer "B.Cu") (net 3))
-  (segment (start 122.428 85.852) (end 122.428 81.788) (width 0.8) (layer "B.Cu") (net 3))
-  (segment (start 126.1872 83.0072) (end 128.524 83.0072) (width 0.8) (layer "B.Cu") (net 3))
   (segment (start 106.38 84.365) (end 103.595 84.365) (width 0.8) (layer "B.Cu") (net 3))
-  (segment (start 124.968 81.788) (end 126.1872 83.0072) (width 0.8) (layer "B.Cu") (net 3))
   (segment (start 102.616 85.344) (end 100.584 85.344) (width 0.8) (layer "B.Cu") (net 3))
+  (segment (start 123.013134 83.0072) (end 128.470105 83.0072) (width 0.8) (layer "B.Cu") (net 3))
   (segment (start 120.101186 88.178814) (end 122.428 85.852) (width 0.8) (layer "B.Cu") (net 3))
-  (segment (start 106.172 84.466823) (end 109.883991 88.178814) (width 0.8) (layer "B.Cu") (net 3))
+  (segment (start 109.883991 88.178814) (end 120.101186 88.178814) (width 0.8) (layer "B.Cu") (net 3))
+  (segment (start 128.470105 83.0072) (end 128.499658 83.036753) (width 0.8) (layer "B.Cu") (net 3))
+  (segment (start 122.428 85.852) (end 122.428 83.592334) (width 0.8) (layer "B.Cu") (net 3))
   (segment (start 103.595 84.365) (end 102.616 85.344) (width 0.8) (layer "B.Cu") (net 3))
-  (segment (start 128.524 85.5472) (end 130.4036 85.5472) (width 0.8) (layer "B.Cu") (net 5))
+  (segment (start 132.08 77.724) (end 134.496 75.308) (width 0.8) (layer "B.Cu") (net 5))
+  (segment (start 130.374047 85.576753) (end 132.08 83.8708) (width 0.8) (layer "B.Cu") (net 5))
+  (segment (start 128.499658 85.576753) (end 130.374047 85.576753) (width 0.8) (layer "B.Cu") (net 5))
+  (segment (start 132.08 83.8708) (end 132.08 77.724) (width 0.8) (layer "B.Cu") (net 5))
+  (segment (start 148.156 75.308) (end 150.368 77.52) (width 0.8) (layer "B.Cu") (net 5))
   (segment (start 134.496 75.308) (end 148.156 75.308) (width 0.8) (layer "B.Cu") (net 5))
-  (segment (start 148.156 75.308) (end 150.368 77.52) (width 0.8) (layer "B.Cu") (net 5))
-  (segment (start 132.08 77.724) (end 134.496 75.308) (width 0.8) (layer "B.Cu") (net 5))
-  (segment (start 130.4036 85.5472) (end 132.08 83.8708) (width 0.8) (layer "B.Cu") (net 5))
-  (segment (start 132.08 83.8708) (end 132.08 77.724) (width 0.8) (layer "B.Cu") (net 5))
+  (segment (start 151.6133 82.2205) (end 153.1373 82.2205) (width 0.8) (layer "B.Cu") (net 6))
+  (segment (start 153.1373 82.2205) (end 154.7368 83.82) (width 0.8) (layer "B.Cu") (net 6))
   (segment (start 154.7368 83.82) (end 160.02 83.82) (width 0.8) (layer "B.Cu") (net 6))
-  (segment (start 151.6133 82.2205) (end 153.1373 82.2205) (width 0.8) (layer "B.Cu") (net 6))
-  (segment (start 138.3912 78.22) (end 147.6128 78.22) (width 0.8) (layer "B.Cu") (net 6))
-  (segment (start 153.1373 82.2205) (end 154.7368 83.82) (width 0.8) (layer "B.Cu") (net 6))
-  (segment (start 136.144 80.4672) (end 138.3912 78.22) (width 0.8) (layer "B.Cu") (net 6))
+  (segment (start 136.119658 80.496753) (end 136.359021 80.496753) (width 0.8) (layer "B.Cu") (net 6))
+  (segment (start 136.359021 80.496753) (end 138.635774 78.22) (width 0.8) (layer "B.Cu") (net 6))
   (segment (start 147.6128 78.22) (end 151.6133 82.2205) (width 0.8) (layer "B.Cu") (net 6))
-  (segment (start 125.476 77.724) (end 125.984 77.216) (width 0.8) (layer "B.Cu") (net 7))
-  (segment (start 125.984 77.216) (end 127.8128 77.216) (width 0.8) (layer "B.Cu") (net 7))
-  (segment (start 127.8128 77.216) (end 128.524 77.9272) (width 0.8) (layer "B.Cu") (net 7))
-  (segment (start 132 91.9188) (end 125.476 85.3948) (width 0.8) (layer "B.Cu") (net 8))
-  (segment (start 132 93.98) (end 132 91.9188) (width 0.8) (layer "B.Cu") (net 8))
-  (segment (start 125.476 85.3948) (end 125.476 85.344) (width 0.8) (layer "B.Cu") (net 8))
+  (segment (start 138.635774 78.22) (end 147.6128 78.22) (width 0.8) (layer "B.Cu") (net 6))
+  (segment (start 125.476 77.724) (end 128.266905 77.724) (width 0.8) (layer "B.Cu") (net 7))
+  (segment (start 128.266905 77.724) (end 128.499658 77.956753) (width 0.8) (layer "B.Cu") (net 7))
+  (segment (start 132 93.98) (end 132 92.884) (width 0.8) (layer "B.Cu") (net 8))
+  (segment (start 132 92.884) (end 125.476 86.36) (width 0.8) (layer "B.Cu") (net 8))
+  (segment (start 125.476 86.36) (end 125.476 85.344) (width 0.8) (layer "B.Cu") (net 8))
+  (segment (start 133.604 86.36) (end 137 89.756) (width 0.8) (layer "B.Cu") (net 9))
+  (segment (start 136.119658 77.956753) (end 135.149247 77.956753) (width 0.8) (layer "B.Cu") (net 9))
+  (segment (start 135.149247 77.956753) (end 133.604 79.502) (width 0.8) (layer "B.Cu") (net 9))
   (segment (start 133.604 79.502) (end 133.604 86.36) (width 0.8) (layer "B.Cu") (net 9))
   (segment (start 137 89.756) (end 137 93.98) (width 0.8) (layer "B.Cu") (net 9))
-  (segment (start 133.604 86.36) (end 137 89.756) (width 0.8) (layer "B.Cu") (net 9))
-  (segment (start 135.1788 77.9272) (end 133.604 79.502) (width 0.8) (layer "B.Cu") (net 9))
-  (segment (start 136.144 77.9272) (end 135.1788 77.9272) (width 0.8) (layer "B.Cu") (net 9))
-  (segment (start 136.144 83.0072) (end 136.652 83.0072) (width 0.8) (layer "B.Cu") (net 10))
+  (segment (start 136.119658 83.036753) (end 136.622447 83.036753) (width 0.8) (layer "B.Cu") (net 10))
+  (segment (start 136.622447 83.036753) (end 138.8872 80.772) (width 0.8) (layer "B.Cu") (net 10))
   (segment (start 138.8872 80.772) (end 139.192 80.772) (width 0.8) (layer "B.Cu") (net 10))
-  (segment (start 136.652 83.0072) (end 138.8872 80.772) (width 0.8) (layer "B.Cu") (net 10))
   (segment (start 146.414 87.0288) (end 148.7842 89.399) (width 0.8) (layer "B.Cu") (net 11))
   (segment (start 161.29 80.8736) (end 158.991 80.8736) (width 0.8) (layer "B.Cu") (net 11))
